Commit message: Updated wheel positions

File: ros/gra_navigation/description/ackermann_macros.xacro (robot description, xacro)
@@ -1,14 +1,14 @@
 <?xml version="1.0"?>
-<robot name="origins" xmlns:xacro="http://www.ros.org/wiki/xacro">
+<robot xmlns:xacro="http://www.ros.org/wiki/xacro" >
     <!-- Constants for math -->
     <xacro:property name="PI" value="3.1415926535897931" />
     <!-- Constants for robot dimensions -->
-    <xacro:property name="length_wheel" value="0.07" />
-    <xacro:property name="radius_wheel" value="0.14" />
-    <xacro:property name="base_center_x" value="0.015" />
-    <xacro:property name="length_from_base_center_to_wheel_x" value="0.395" />
-    <xacro:property name="length_from_base_to_wheel_front_x" value="0.41" />
-    <xacro:property name="length_from_base_to_wheel_rear_x" value="0.38" />
-    <xacro:property name="length_from_base_to_wheel_y" value="0.25" />
+    <xacro:property name="length_wheel" value="0.2" />
+    <xacro:property name="radius_wheel" value="0.25" />
+    <xacro:property name="base_center_x" value="0" />
+    <xacro:property name="length_from_base_center_to_wheel_x" value="0.77" /> <!-- this is the distance between front wheel and rear wheel divided by 2 -->
+    <xacro:property name="length_from_base_to_wheel_front_x" value="0.77" />
+    <xacro:property name="length_from_base_to_wheel_rear_x" value="0.77" />
+    <xacro:property name="length_from_base_to_wheel_y" value="0.6" />
     <xacro:macro name="default_inertial" params="mass">
         <inertial>
@@ -36,13 +36,18 @@
         </joint>
     </xacro:macro>
+    <gazebo>
+        <plugin name="gazebo_ros_control" filename="libgazebo_ros_control.so">
+        </plugin>
+    </gazebo>
     <xacro:macro name="wheel" params="right_left reflect_right_left front_rear reflect_front_rear">
         <link name="${right_left}_${front_rear}_wheel">
             <visual>
                 <!-- when reflect_right_left = 1 to be 0 reflect_right_left= -1 to be PI -->
-                <origin rpy="${PI/2-reflect_right_left*PI/2} 0 0" xyz="0 0 0"/>
+                <origin rpy="${PI/2} 0 0" xyz="0 0 0"/>
                 <!-- <origin rpy="${PI/2-reflect_right_left*PI/2} 0 0" xyz="0 0 0"/> -->
                 <geometry>
-                    <mesh filename="package://cirkit_unit03_description/meshes/cirkit_unit03/cirkit_unit03_wheel.dae"/>
+                    <cylinder length="${length_wheel}" radius="${radius_wheel}" />
                 </geometry>
+                <material name="black"/>
             </visual>
             <collision>
@@ -86,5 +91,5 @@
             <parent link="base_link"/>
             <child link="steer_${right_left}"/>
-            <origin xyz="${base_center_x+length_from_base_center_to_wheel_x} ${-reflect_right_left*length_from_base_to_wheel_y} 0.30"/>
+            <origin xyz="${base_center_x+length_from_base_center_to_wheel_x} ${-reflect_right_left*length_from_base_to_wheel_y} ${radius_wheel}"/>
             <dynamics damping="0.7" friction="0.7"/>
             <limit effort="7.0" lower="${-80*PI/180}" upper="${80*PI/180}" velocity="${200.0*PI/180.0*0.95}"/>
@@ -93,9 +98,10 @@
             <visual>
                 <!-- when reflect_right_left = 1 to be 0 reflect_right_left= -1 to be PI -->
-                <origin rpy="${PI/2-reflect_right_left*PI/2} 0 0" xyz="0 0 0"/>
+                <origin rpy="${PI/2} 0 0" xyz="0 0 0"/>
                 <!-- <origin rpy="${PI/2-reflect_right_left*PI/2} 0 0" xyz="0 0 0"/> -->
                 <geometry>
-                    <mesh filename="package://cirkit_unit03_description/meshes/cirkit_unit03/cirkit_unit03_wheel.dae"/>
+                    <cylinder length="${length_wheel}" radius="${radius_wheel}" />
                 </geometry>
+                <material name="black"/>
             </visual>
             <collision>
@@ -112,5 +118,5 @@
             <child link="${right_left}_front_wheel"/>
             <!-- <origin xyz="${base_center_x+length_from_base_center_to_wheel_x} ${-reflect_right_left*length_from_base_to_wheel_y} ${radius_wheel}"/> -->
-            <origin xyz="0 0 -0.16"/>
+            <origin xyz="0 0 0"/>
         </joint>
         <transmission name="tran_${right_left}_front">

File: ros/gra_navigation/description/robot_core.xacro (robot description, xacro)
@@ -52,192 +52,40 @@
         <material>Gazebo/White</material>
     </gazebo>
-    <!-- WHEEL 1 (CLOCKWISE) -->
-    <joint name="wheel_1_joint" type="continuous">
+    <xacro:rear_wheel/>
+    <xacro:front_wheel right_left="right" reflect_right_left="1"/>
+    <xacro:front_wheel right_left="left" reflect_right_left="-1"/>
+    <xacro:wheel right_left="right" reflect_right_left="1" front_rear="rear" reflect_front_rear="-1"/>
+    <xacro:wheel right_left="left" reflect_right_left="-1" front_rear="rear" reflect_front_rear="-1"/>
+    <!-- steer -->
+    <link name="front_steer_link"/>
+    <joint name="front_steer_joint" type="fixed">
+        <axis xyz="0 1 0"/>
         <parent link="base_link"/>
-        <child link="wheel_1"/>
-        <origin xyz="1.25 0.5 0.2" rpy="${pi/2} 0 0"/>
-        <axis xyz="0 0 1"/>
+        <child link="front_steer_link"/>
+        <origin xyz="0.77 0 0.25"/>
     </joint>
-    <link name="wheel_1">
-        <visual>
-            <geometry>
-                <cylinder length="0.25" radius="0.20" />
-            </geometry>
-            <material name="black"/>
-        </visual>
-        <collision>
-            <geometry>
-                <cylinder length="0.25" radius="0.20" />
-            </geometry>
-        </collision>
-        <xacro:inertial_cylinder mass="5" length="0.25" radius="0.20">
-            <origin xyz="0 0 0" rpy="0 0 0"/>
-        </xacro:inertial_cylinder>
-    </link>
-    <gazebo reference="wheel_1">
-        <material>Gazebo/Black</material>
-        <mu1 value="0.2"/>
-        <mu2 value="1.5"/>
-        <kp value="10000000.0" />
-        <kd value="10000.0" />
-        <fdir1 value="0 0 1"/>
-        <maxContacts value= "1"/>
-    </gazebo>
-    <!-- WHEEL 2 -->
-    <joint name="wheel_2_joint" type="continuous">
-        <parent link="base_link"/>
-        <child link="wheel_2"/>
-        <origin xyz="1.25 -0.5 0.2" rpy="-${pi/2} 0 0"/>
-        <axis xyz="0 0 1"/>
-    </joint>
-    <link name="wheel_2">
-        <visual>
-            <geometry>
-                <cylinder length="0.25" radius="0.20" />
-            </geometry>
-            <material name="black"/>
-        </visual>
-        <collision>
-            <geometry>
-                <cylinder length="0.25" radius="0.20" />
-            </geometry>
-        </collision>
-        <xacro:inertial_cylinder mass="5" length="0.25" radius="0.20">
-            <origin xyz="0 0 0" rpy="0 0 0"/>
-        </xacro:inertial_cylinder>
-    </link>
-    <gazebo reference="wheel_2">
-        <material>Gazebo/Black</material>
-        <mu1 value="0.2"/>
-        <mu2 value="1.5"/>
-        <kp value="10000000.0" />
-        <kd value="10000.0" />
-        <fdir1 value="0 0 1"/>
-        <maxContacts value= "1"/>
-    </gazebo>
-    <!-- WHEEL 3 -->
-    <joint name="wheel_3_joint" type="continuous">
-        <parent link="base_link"/>
-        <child link="wheel_3"/>
-        <origin xyz="-1.25 -0.5 0.2" rpy="-${pi/2} 0 0"/>
-        <axis xyz="0 0 1"/>
-    </joint>
-    <link name="wheel_3">
-        <visual>
-            <geometry>
-                <cylinder length="0.25" radius="0.20" />
-            </geometry>
-            <material name="black"/>
-        </visual>
-        <collision>
-            <geometry>
-                <cylinder length="0.25" radius="0.20" />
-            </geometry>
-        </collision>
-        <xacro:inertial_cylinder mass="5" length="0.25" radius="0.20">
-            <origin xyz="0 0 0" rpy="0 0 0"/>
-        </xacro:inertial_cylinder>
-    </link>
-    <gazebo reference="wheel_3">
-        <material>Gazebo/Black</material>
-        <mu1 value="0.2"/>
-        <mu2 value="1.5"/>
-        <kp value="10000000.0" />
-        <kd value="10000.0" />
-        <fdir1 value="0 0 1"/>
-        <maxContacts value= "1"/>
-    </gazebo>
-        <!-- WHEEL 4 -->
-    <joint name="wheel_4_joint" type="continuous">
-        <parent link="base_link"/>
-        <child link="wheel_4"/>
-        <origin xyz="-1.25 0.5 0.2" rpy="${pi/2} 0 0"/>
-        <axis xyz="0 0 1"/>
-    </joint>
-    <link name="wheel_4">
-        <visual>
-            <geometry>
-                <cylinder length="0.25" radius="0.20" />
-            </geometry>
-            <material name="black"/>
-        </visual>
-        <collision>
-            <geometry>
-                <cylinder length="0.25" radius="0.20" />
-            </geometry>
-        </collision>
-        <xacro:inertial_cylinder mass="5" length="0.25" radius="0.20">
-            <origin xyz="0 0 0" rpy="0 0 0"/>
-        </xacro:inertial_cylinder>
-    </link>
-    <gazebo reference="wheel_4">
-        <material>Gazebo/Black</material>
-        <mu1 value="0.2"/>
-        <mu2 value="1.5"/>
-        <kp value="10000000.0" />
-        <kd value="10000.0" />
-        <fdir1 value="0 0 1"/>
-        <maxContacts value= "1"/>
-    </gazebo>
-    <!-- Joint for wheel_1 (left front wheel) steering -->
-    <joint name="wheel_1_steer_joint" type="revolute">
-        <parent link="base_link"/>
-        <child link="wheel_1"/>
-        <origin xyz="1.25 0.5 0.2" rpy="${pi/2} 0 0"/> <!-- adjust xyz as needed -->
-        <axis xyz="0 1 0"/>
-        <limit lower="-0.7854" upper="0.7854" effort="100" velocity="1"/> <!-- -45 to 45 degrees in radians -->
-    </joint>
-    <!-- Joint for wheel_2 (right front wheel) steering -->
-    <joint name="wheel_2_steer_joint" type="revolute">
-        <parent link="base_link"/>
-        <child link="wheel_2"/>
-        <origin xyz="1.25 -0.5 0.2" rpy="-${pi/2} 0 0"/> <!-- adjust xyz as needed -->
-        <axis xyz="0 1 0"/>
-        <limit lower="-0.7854" upper="0.7854" effort="100" velocity="1"/> <!-- -45 to 45 degrees in radians -->
-    </joint>
-    <!-- Transmissions -->
     <transmission name="tran1">
-        <type>transmission_interface/SimpleTransmission</type>
-        <joint name="wheel_1_joint">
-            <hardwareInterface>hardware_interface/VelocityJointInterface</hardwareInterface>
+      <type>transmission_interface/SimpleTransmission</type>
+        <joint name="base_to_left_rear_wheel">
+          <hardwareInterface>EffortJointInterface</hardwareInterface>
         </joint>
-        <actuator name="motor_1">
-            <hardwareInterface>VelocityJointInterface</hardwareInterface>
-            <mechanicalReduction>1</mechanicalReduction>
+        <actuator name="motor1">
+          <hardwareInterface>EffortJointInterface</hardwareInterface>
+          <mechanicalReduction>1</mechanicalReduction>
         </actuator>
     </transmission>
     <transmission name="tran2">
-        <type>transmission_interface/SimpleTransmission</type>
-        <joint name="wheel_2_joint">
-            <hardwareInterface>hardware_interface/VelocityJointInterface</hardwareInterface>
-        </joint>
-        <actuator name="motor_2">
-            <hardwareInterface>VelocityJointInterface</hardwareInterface>
-            <mechanicalReduction>1</mechanicalReduction>
-        </actuator>
+      <type>transmission_interface/SimpleTransmission</type>
+      <joint name="base_to_right_rear_wheel">
+        <hardwareInterface>EffortJointInterface</hardwareInterface>
+      </joint>
+      <actuator name="motor2">
+        <hardwareInterface>EffortJointInterface</hardwareInterface>
+        <mechanicalReduction>1</mechanicalReduction>
+      </actuator>
     </transmission>
-    <transmission name="tran3">
-        <type>transmission_interface/SimpleTransmission</type>
-        <joint name="wheel_3_joint">
-            <hardwareInterface>hardware_interface/VelocityJointInterface</hardwareInterface>
-        </joint>
-        <actuator name="motor_3">
-            <hardwareInterface>VelocityJointInterface</hardwareInterface>
-            <mechanicalReduction>1</mechanicalReduction>
-        </actuator>
-    </transmission>
-    <transmission name="tran4">
-        <type>transmission_interface/SimpleTransmission</type>
-        <joint name="wheel_4_joint">
-            <hardwareInterface>hardware_interface/VelocityJointInterface</hardwareInterface>
-        </joint>
-        <actuator name="motor_4">
-            <hardwareInterface>VelocityJointInterface</hardwareInterface>
-            <mechanicalReduction>1</mechanicalReduction>
-        </actuator>
-    </transmission>
-    <gazebo>
+    <!-- <gazebo>
         <plugin name="gazebo_ros_control" filename="libgazebo_ros_control.so">
         </plugin>
-    </gazebo>
+    </gazebo> -->
 </robot>

Commit message: updated robotHW for ackermann
not working

File: ros/gra_navigation/description/ackermann_macros.xacro (robot description, xacro)
@@ -93,5 +93,5 @@
             <origin xyz="${base_center_x+length_from_base_center_to_wheel_x} ${-reflect_right_left*length_from_base_to_wheel_y} ${radius_wheel}"/>
             <dynamics damping="0.7" friction="0.7"/>
-            <limit effort="7.0" lower="${-80*PI/180}" upper="${80*PI/180}" velocity="${200.0*PI/180.0*0.95}"/>
+            <limit effort="7.0" lower="${-45*PI/180}" upper="${45*PI/180}" velocity="${200.0*PI/180.0*0.95}"/>
         </joint>
         <link name="${right_left}_front_wheel">
